Commit message: Enhance robot description: add gripper functionality and update URDF dimensions

File: urdf/6dof-robot.urdf (robot description, URDF)
Before this commit: robot rough_6dof_arm, 8 links, 7 joints
Links:
- added link gripper_base_link, mass 0.20; collision cylinder length=0.015 radius=0.035; visual cylinder length=0.015 radius=0.035
- added link gripper_command_link
- added link left_finger_link, mass 0.04; collision box size=0.030 0.008 0.012; visual box size=0.030 0.008 0.012
- added link right_finger_link, mass 0.04; collision box size=0.030 0.008 0.012; visual box size=0.030 0.008 0.012
Joints:
- added joint gripper_joint: type revolute, parent gripper_base_link, child gripper_command_link, origin xyz=0 0 0 rpy=0 0 0, axis 1 0 0, limit lower=0 upper=3.14159265359 effort=20 velocity=2.0
- added joint gripper_mount_joint: type fixed, parent tool_link, child gripper_base_link, origin xyz=0.090 0 0 rpy=0 0 0
- added joint left_finger_joint: type prismatic, parent gripper_base_link, child left_finger_link, origin xyz=0 0 0 rpy=0 0 0, axis 0 1 0, limit lower=0 upper=0.020 effort=20 velocity=0.05, mimic joint=gripper_joint multiplier=0.006366197724 offset=0
- added joint right_finger_joint: type prismatic, parent gripper_base_link, child right_finger_link, origin xyz=0 0 0 rpy=0 0 0, axis 0 -1 0, limit lower=0 upper=0.020 effort=20 velocity=0.05, mimic joint=gripper_joint multiplier=0.006366197724 offset=0
- joint tcp_fixed_joint: origin xyz=0.090 0 0 rpy=0 0 0 -> xyz=0.015 0 0 rpy=0 0 0; parent tool_link -> gripper_base_link

Commit message: Update URDF joint limits and README for accuracy based on firmware specifications

File: urdf/6dof-robot.urdf (robot description, URDF)
Before this commit: robot rough_6dof_arm, 12 links, 11 joints
Joints:
- joint joint_1: limit lower=-3.14159 upper=3.14159 effort=100 velocity=1.5 -> lower=-1.65806278939 upper=1.65806278939 effort=100 velocity=1.5
- joint joint_2: limit lower=-2.61799 upper=2.61799 effort=100 velocity=1.5 -> lower=-1.30899693900 upper=1.22173047640 effort=100 velocity=1.5
- joint joint_3: limit lower=-2.61799 upper=2.61799 effort=80 velocity=1.8 -> lower=-0.872664625997 upper=0.942477796077 effort=80 velocity=1.8
- joint joint_4: limit lower=-3.14159 upper=3.14159 effort=35 velocity=2.5 -> lower=-2.79252680319 upper=2.79252680319 effort=35 velocity=2.5
- joint joint_5: limit lower=-2.61799 upper=2.61799 effort=30 velocity=2.5 -> lower=-1.74532925199 upper=1.74532925199 effort=30 velocity=2.5
- joint joint_6: limit lower=-3.14159 upper=3.14159 effort=25 velocity=3.0 -> lower=-2.09439510239 upper=2.09439510239 effort=25 velocity=3.0

Commit message: Fix joint axis orientations in URDF for correct kinematics

File: urdf/6dof-robot.urdf (robot description, URDF)
Before this commit: robot rough_6dof_arm, 12 links, 11 joints
Joints:
- joint joint_1: axis 0 0 1 -> 0 0 -1
- joint joint_2: axis 0 1 0 -> 0 -1 0
- joint joint_4: axis 1 0 0 -> -1 0 0
- joint joint_5: axis 0 1 0 -> 0 -1 0
- joint joint_6: axis 1 0 0 -> -1 0 0
